Commit message: Update my_robot.xacro
change robot color

File: P2-Go-Chase-It/catkin_ws/src/my_robot/urdf/my_robot.xacro (robot description, xacro)
@@ -24,4 +24,7 @@
         <box size=".4 .2 .1"/>
       </geometry>
+      <material name="black_metal">
+        <color rgba="1 0 0 1"/>
+      </material>
     </collision>
     <visual name='chassis_visual'>
@@ -184,3 +187,15 @@
     <dynamics damping="1.0" friction="1.0"/>
   </joint>
+  <gazebo reference="chassis">
+    <material>Gazebo/Green</material>
+  </gazebo>
+  <gazebo reference="left_wheel">
+    <material>Gazebo/Blue</material>
+  </gazebo>
+  <gazebo reference="right_wheel">
+    <material>Gazebo/Blue</material>
+  </gazebo>
+  <gazebo reference="camera">
+    <material>Gazebo/Red</material>
+  </gazebo>
 </robot>
